File: CFA/CFA.sch (EAGLE design)
At the start: 77 parts, among them IC1 OPA345P, Q1 BC550C, Q10 BC560C, Q11 BC550C, Q12 MJE15030, Q13 MJE15031, Q14 MJE15030, Q15 BC560C, Q16 MJE15031, Q17 MJE15031, Q18 BC560C, Q19 BC550C, Q2 BC550C, Q20 BC550C, Q21 MJE15030, Q22 BC560C, Q23 BC560C, Q24 BC550C, Q25 BC550C, Q27 PZTA56, Q28 PZTA06SOT-223, Q3 BC560C, Q4 BC560C, Q5 MJE15030, Q6 BC560C, Q7 BC550C, Q8 BC550C, Q9 BC560C, X1 MKDSN1,5/2-5,08, X2 MKDSN1,5/2-5,08

Commit message: VCFA2
Connections:
- net N$1: now also Q21.B, R30.1; no longer Q21.E
- net N$48: now also Q21.E; no longer Q21.B, R30.1
Changed lines of the file:
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@@
 <?xml version="1.0" encoding="utf-8"?>
 <!DOCTYPE eagle SYSTEM "eagle.dtd">
-<eagle version="9.3.1">
+<eagle version="9.4.2">
 <drawing>
 <settings>
-<setting alwaysvectorfont="yes"/>
+<setting alwaysvectorfont="no"/>
 <setting verticaltext="up"/>
 </settings>
@@
 <net name="N$48" class="0">
 <segment>
-<pinref part="Q21" gate="1" pin="B"/>
-<wire x1="149.86" y1="106.68" x2="144.78" y2="106.68" width="0.1524" layer="91"/>
-<pinref part="R30" gate="G$1" pin="1"/>
-<wire x1="144.78" y1="111.76" x2="144.78" y2="106.68" width="0.1524" layer="91"/>
-<junction x="144.78" y="106.68"/>
-<wire x1="144.78" y1="106.68" x2="144.78" y2="96.52" width="0.1524" layer="91"/>
-<wire x1="144.78" y1="96.52" x2="154.94" y2="96.52" width="0.1524" layer="91"/>
 <pinref part="R15" gate="G$1" pin="2"/>
 <wire x1="149.86" y1="60.96" x2="149.86" y2="63.5" width="0.1524" layer="91"/>
@@
 <wire x1="149.86" y1="63.5" x2="154.94" y2="63.5" width="0.1524" layer="91"/>
 <junction x="154.94" y="63.5"/>
-<wire x1="154.94" y1="96.52" x2="154.94" y2="86.36" width="0.1524" layer="91"/>
+<wire x1="154.94" y1="101.6" x2="154.94" y2="86.36" width="0.1524" layer="91"/>
 <junction x="154.94" y="86.36"/>
+<pinref part="Q21" gate="1" pin="E"/>
 </segment>
 </net>
@@
 <pinref part="C7" gate="G$1" pin="1"/>
 <junction x="137.16" y="-17.78"/>
-<pinref part="C7" gate="G$1" pin="1"/>
 </segment>
 <segment>
@@
 <pinref part="C6" gate="G$1" pin="1"/>
 <junction x="137.16" y="-2.54"/>
-<pinref part="C6" gate="G$1" pin="1"/>
 </segment>
 <segment>
@@
 <segment>
 <pinref part="RV1" gate="G$1" pin="E"/>
-<wire x1="144.78" y1="91.44" x2="144.78" y2="93.98" width="0.1524" layer="91"/>
-<wire x1="144.78" y1="93.98" x2="160.02" y2="93.98" width="0.1524" layer="91"/>
-<wire x1="160.02" y1="93.98" x2="160.02" y2="101.6" width="0.1524" layer="91"/>
-<pinref part="Q21" gate="1" pin="E"/>
-<wire x1="160.02" y1="101.6" x2="154.94" y2="101.6" width="0.1524" layer="91"/>
-</segment>
-</net>
+<pinref part="Q21" gate="1" pin="B"/>
+<wire x1="149.86" y1="106.68" x2="144.78" y2="106.68" width="0.1524" layer="91"/>
+<pinref part="R30" gate="G$1" pin="1"/>
+<wire x1="144.78" y1="111.76" x2="144.78" y2="106.68" width="0.1524" layer="91"/>
+<wire x1="144.78" y1="91.44" x2="144.78" y2="106.68" width="0.1524" layer="91"/>
+<junction x="144.78" y="106.68"/>
+</segment>
+</net>
