File: CFA/CFA_c.brd (EAGLE design)
At the start: 109.2 x 116.5 mm, 192 parts, among them IC1 OPA2132U, IC3 OPA2132U, Q1 BC847CSMD, Q10 BC857CSMD, Q11 BC847CSMD, Q12 MJE15030, Q13 MJE15031, Q14 MJE15030, Q15 BC857CSMD, Q16 MJE15031, Q17 MJE15031, Q18 BC857CSMD, Q19 BC847CSMD, Q2 BC847CSMD, Q20 BC847CSMD, Q21 MJE15030, Q22 BC857CSMD, Q23 BC857CSMD, Q24 BC847CSMD, Q25 BC847CSMD, Q26 BC847CSMD, Q27 PZTA56, Q28 PZTA06SOT-223, Q29 BC857CSMD, Q3 BC857CSMD, Q30 BC847CSMD, Q31 BC847CSMD, Q32 BC847CSMD, Q33 BC857CSMD, Q34 BC857CSMD, Q35 BC857CSMD, Q36 BC857CSMD, Q37 BC847CSMD, Q38 BC847CSMD, Q39 BC847CSMD, Q4 BC857CSMD, Q40 BC857CSMD, Q41 BC857CSMD, Q5 MJE15030, Q55 BC847CSMD, Q56 BC847CSMD, Q57 BC857CSMD, Q58 BC857CSMD, Q59 MJE15030, Q6 BC857CSMD, Q60 MJE15031, Q61 BC847CSMD, Q62 BC857CSMD, Q63 BC857CSMD, Q64 BC847CSMD, Q65 BC857CSMD, Q66 BC857CSMD, Q67 PZTA56, Q68 MJE15030, Q69 MJE15031, Q7 BC847CSMD, Q70 MJE15030, Q71 MJE15031, Q72 BC847CSMD, Q73 BC847CSMD, Q74 MJE15030, Q75 BC857CSMD, Q76 BC857CSMD, Q77 BC847CSMD, Q78 BC847CSMD, Q79 PZTA06SOT-223, Q8 BC847CSMD, Q80 BC857CSMD, Q81 BC847CSMD, Q9 BC857CSMD

Commit message: VCFA2
Connections:
- removed net N$231: Q74.3, RV3.3
- new net N$122: Q74.1, R90.1, RV3.3
- net N$1: now also Q21.1, R30.1; no longer Q21.3
- net N$223: now also Q74.3; no longer Q74.1, R90.1
- net N$48: now also Q21.3; no longer Q21.1, R30.1
Routing:
- net N$231: track 14.5 -> 0.00 mm, vias 2 -> 0
- net N$48: track 58.0 -> 49.6 mm
- net N$223: track 58.0 -> 49.6 mm
- net N$1: track 14.5 -> 13.7 mm
Changed lines of the file:
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@@
 </signal>
 <signal name="N$48">
-<contactref element="Q21" pad="1"/>
-<contactref element="R30" pad="1"/>
 <contactref element="R15" pad="2"/>
 <contactref element="Q28" pad="2"/>
@@
 <wire x1="26.787" y1="30.363" x2="26.198" y2="30.363" width="0.6096" layer="1"/>
 <wire x1="29.337" y1="27.813" x2="26.787" y2="30.363" width="0.6096" layer="1"/>
-<wire x1="26.821" y1="33.401" x2="26.821" y2="30.397" width="0.6096" layer="1"/>
 <wire x1="26.821" y1="30.397" x2="26.787" y2="30.363" width="0.6096" layer="1"/>
 <wire x1="27.498" y1="36.195" x2="26.821" y2="35.518" width="0.6096" layer="1"/>
-<wire x1="26.821" y1="35.518" x2="26.821" y2="33.401" width="0.6096" layer="1"/>
 <wire x1="30.698" y1="27.813" x2="30.698" y2="26.888" width="0.6096" layer="1"/>
 <wire x1="26.921" y1="23.111" x2="26.921" y2="21.844" width="0.6096" layer="1"/>
 <wire x1="30.698" y1="26.888" x2="26.921" y2="23.111" width="0.6096" layer="1"/>
 <wire x1="35.56" y1="35.56" x2="32.969" y2="35.56" width="1.016" layer="1"/>
-<wire x1="37.87" y1="30.22" x2="35.56" y2="32.53" width="1.016" layer="1"/>
 <wire x1="35.56" y1="32.53" x2="35.56" y2="35.56" width="1.016" layer="1"/>
 <wire x1="43.44" y1="41.68" x2="41.148" y2="39.388" width="1.016" layer="1"/>
@@
 <wire x1="27.686" y1="34.925" x2="27.498" y2="35.113" width="0.508" layer="1"/>
 <wire x1="39.167" y1="35.56" x2="35.56" y2="35.56" width="1.016" layer="1"/>
+<contactref element="Q21" pad="3"/>
+<wire x1="35.56" y1="32.53" x2="37.87" y2="25.66" width="0" layer="19" extent="1-1"/>
+<wire x1="26.821" y1="30.397" x2="27.686" y2="34.925" width="0" layer="19" extent="1-1"/>
 </signal>
 <signal name="N$35">
@@
 <wire x1="15.494" y1="33.02" x2="15.24" y2="33.02" width="0.508" layer="16"/>
 </signal>
-<signal name="N$1">
-<contactref element="RV1" pad="3"/>
-<contactref element="Q21" pad="3"/>
-<wire x1="26.198" y1="25.263" x2="26.67" y2="25.735" width="0.6096" layer="1"/>
-<wire x1="26.67" y1="25.735" x2="26.67" y2="26.67" width="0.6096" layer="1"/>
-<via x="26.67" y="26.67" extent="1-16" drill="0.35"/>
-<wire x1="26.67" y1="26.67" x2="33.02" y2="26.67" width="0.6096" layer="16"/>
-<wire x1="33.02" y1="26.67" x2="35.56" y2="24.13" width="0.6096" layer="16"/>
-<via x="35.56" y="24.13" extent="1-16" drill="0.35"/>
-<wire x1="35.56" y1="24.13" x2="37.09" y2="25.66" width="0.6096" layer="1"/>
-<wire x1="37.09" y1="25.66" x2="37.87" y2="25.66" width="0.6096" layer="1"/>
-</signal>
 <signal name="N$17">
 <contactref element="C1" pad="1"/>
@@
 </signal>
 <signal name="N$223">
-<contactref element="Q74" pad="1"/>
-<contactref element="R90" pad="1"/>
 <contactref element="R78" pad="2"/>
 <contactref element="Q79" pad="2"/>
@@
 <wire x1="26.787" y1="87.513" x2="26.198" y2="87.513" width="0.6096" layer="1"/>
 <wire x1="29.337" y1="84.963" x2="26.787" y2="87.513" width="0.6096" layer="1"/>
-<wire x1="26.821" y1="90.551" x2="26.821" y2="87.547" width="0.6096" layer="1"/>
 <wire x1="26.821" y1="87.547" x2="26.787" y2="87.513" width="0.6096" layer="1"/>
 <wire x1="27.498" y1="93.345" x2="26.821" y2="92.668" width="0.6096" layer="1"/>
-<wire x1="26.821" y1="92.668" x2="26.821" y2="90.551" width="0.6096" layer="1"/>
 <wire x1="30.698" y1="84.963" x2="30.698" y2="84.038" width="0.6096" layer="1"/>
 <wire x1="26.921" y1="80.261" x2="26.921" y2="78.994" width="0.6096" layer="1"/>
 <wire x1="30.698" y1="84.038" x2="26.921" y2="80.261" width="0.6096" layer="1"/>
 <wire x1="35.56" y1="92.71" x2="32.969" y2="92.71" width="1.016" layer="1"/>
-<wire x1="37.87" y1="87.37" x2="35.56" y2="89.68" width="1.016" layer="1"/>
 <wire x1="35.56" y1="89.68" x2="35.56" y2="92.71" width="1.016" layer="1"/>
 <wire x1="43.44" y1="98.83" x2="41.148" y2="96.538" width="1.016" layer="1"/>
@@
 <wire x1="27.686" y1="92.075" x2="27.498" y2="92.263" width="0.508" layer="1"/>
 <wire x1="39.167" y1="92.71" x2="35.56" y2="92.71" width="1.016" layer="1"/>
+<contactref element="Q74" pad="3"/>
+<wire x1="26.821" y1="87.547" x2="27.686" y2="92.075" width="0" layer="19" extent="1-1"/>
+<wire x1="37.87" y1="82.81" x2="35.56" y2="89.68" width="0" layer="19" extent="1-1"/>
 </signal>
 <signal name="N$224">
@@
 <wire x1="15.494" y1="90.17" x2="15.24" y2="90.17" width="0.508" layer="16"/>
 </signal>
-<signal name="N$231">
-<contactref element="RV3" pad="3"/>
-<contactref element="Q74" pad="3"/>
-<wire x1="26.198" y1="82.413" x2="26.67" y2="82.885" width="0.6096" layer="1"/>
-<wire x1="26.67" y1="82.885" x2="26.67" y2="83.82" width="0.6096" layer="1"/>
-<via x="26.67" y="83.82" extent="1-16" drill="0.35"/>
-<wire x1="26.67" y1="83.82" x2="33.02" y2="83.82" width="0.6096" layer="16"/>
-<wire x1="33.02" y1="83.82" x2="35.56" y2="81.28" width="0.6096" layer="16"/>
-<via x="35.56" y="81.28" extent="1-16" drill="0.35"/>
-<wire x1="35.56" y1="81.28" x2="37.09" y2="82.81" width="0.6096" layer="1"/>
-<wire x1="37.09" y1="82.81" x2="37.87" y2="82.81" width="0.6096" layer="1"/>
-</signal>
 <signal name="N$232">
 <contactref element="C18" pad="1"/>
@@
 <wire x1="-30.48" y1="42.39" x2="-34.29" y2="42.14" width="0" layer="19" extent="1-1"/>
 </signal>
+<signal name="N$122">
+<contactref element="Q74" pad="1"/>
+<contactref element="R90" pad="1"/>
+<contactref element="RV3" pad="3"/>
+<wire x1="26.821" y1="90.551" x2="37.87" y2="87.37" width="0" layer="19" extent="1-1"/>
+<wire x1="26.198" y1="82.413" x2="26.821" y2="90.551" width="0" layer="19" extent="1-1"/>
+</signal>
+<signal name="N$1">
+<contactref element="Q21" pad="1"/>
+<contactref element="R30" pad="1"/>
+<contactref element="RV1" pad="3"/>
+<wire x1="26.198" y1="25.263" x2="26.67" y2="25.735" width="0.6096" layer="1"/>
+<wire x1="26.67" y1="25.735" x2="26.67" y2="26.67" width="0.6096" layer="1"/>
+<via x="26.67" y="26.67" extent="1-16" drill="0.35"/>
+<wire x1="26.67" y1="26.67" x2="33.02" y2="26.67" width="0.6096" layer="16"/>
+<wire x1="33.02" y1="26.67" x2="35.56" y2="24.13" width="0.6096" layer="16"/>
+<via x="35.56" y="24.13" extent="1-16" drill="0.35"/>
+<wire x1="35.56" y1="24.13" x2="37.09" y2="25.66" width="0.6096" layer="1"/>
+<wire x1="37.09" y1="25.66" x2="37.87" y2="30.22" width="0" layer="19" extent="1-1"/>
+<wire x1="26.821" y1="33.401" x2="26.67" y2="26.67" width="0" layer="19" extent="1-16"/>
+</signal>
 </signals>
