File: CFA/CFA_c.sch (EAGLE design)
At the start: 192 parts, among them IC1 OPA2132U, IC3 OPA2132U, Q1 BC847CSMD, Q10 BC857CSMD, Q11 BC847CSMD, Q12 MJE15030, Q13 MJE15031, Q14 MJE15030, Q15 BC857CSMD, Q16 MJE15031, Q17 MJE15031, Q18 BC857CSMD, Q19 BC847CSMD, Q2 BC847CSMD, Q20 BC847CSMD, Q21 MJE15030, Q22 BC857CSMD, Q23 BC857CSMD, Q24 BC847CSMD, Q25 BC847CSMD, Q26 BC847CSMD, Q27 PZTA56, Q28 PZTA06SOT-223, Q29 BC857CSMD, Q3 BC857CSMD, Q30 BC847CSMD, Q31 BC847CSMD, Q32 BC847CSMD, Q33 BC857CSMD, Q34 BC857CSMD, Q35 BC857CSMD, Q36 BC857CSMD, Q37 BC847CSMD, Q38 BC847CSMD, Q39 BC847CSMD, Q4 BC857CSMD, Q40 BC857CSMD, Q41 BC857CSMD, Q5 MJE15030, Q55 BC847CSMD, Q56 BC847CSMD, Q57 BC857CSMD, Q58 BC857CSMD, Q59 MJE15030, Q6 BC857CSMD, Q60 MJE15031, Q61 BC847CSMD, Q62 BC857CSMD, Q63 BC857CSMD, Q64 BC847CSMD, Q65 BC857CSMD, Q66 BC857CSMD, Q67 PZTA56, Q68 MJE15030, Q69 MJE15031, Q7 BC847CSMD, Q70 MJE15030, Q71 MJE15031, Q72 BC847CSMD, Q73 BC847CSMD, Q74 MJE15030, Q75 BC857CSMD, Q76 BC857CSMD, Q77 BC847CSMD, Q78 BC847CSMD, Q79 PZTA06SOT-223, Q8 BC847CSMD, Q80 BC857CSMD, Q81 BC847CSMD, Q9 BC857CSMD

Commit message: VCFA2
Connections:
- removed net N$231: Q74.E, RV3.E
- new net N$122: Q74.B, R90.1, RV3.E
- net N$1: now also Q21.B, R30.1; no longer Q21.E
- net N$223: now also Q74.E; no longer Q74.B, R90.1
- net N$48: now also Q21.E; no longer Q21.B, R30.1
Changed lines of the file:
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@@
 <net name="N$48" class="0">
 <segment>
-<pinref part="Q21" gate="G$1" pin="B"/>
-<wire x1="149.86" y1="106.68" x2="144.78" y2="106.68" width="0.1524" layer="91"/>
-<pinref part="R30" gate="G$1" pin="1"/>
-<wire x1="144.78" y1="111.76" x2="144.78" y2="106.68" width="0.1524" layer="91"/>
-<junction x="144.78" y="106.68"/>
-<wire x1="144.78" y1="106.68" x2="144.78" y2="96.52" width="0.1524" layer="91"/>
-<wire x1="144.78" y1="96.52" x2="154.94" y2="96.52" width="0.1524" layer="91"/>
 <pinref part="R15" gate="G$1" pin="2"/>
 <wire x1="149.86" y1="60.96" x2="149.86" y2="63.5" width="0.1524" layer="91"/>
@@
 <wire x1="149.86" y1="63.5" x2="154.94" y2="63.5" width="0.1524" layer="91"/>
 <junction x="154.94" y="63.5"/>
-<wire x1="154.94" y1="96.52" x2="154.94" y2="86.36" width="0.1524" layer="91"/>
+<wire x1="154.94" y1="101.6" x2="154.94" y2="86.36" width="0.1524" layer="91"/>
 <junction x="154.94" y="86.36"/>
+<pinref part="Q21" gate="G$1" pin="E"/>
 </segment>
 </net>
@@
 </segment>
 </net>
-<net name="N$1" class="0">
-<segment>
-<pinref part="RV1" gate="G$1" pin="E"/>
-<wire x1="144.78" y1="91.44" x2="144.78" y2="93.98" width="0.1524" layer="91"/>
-<wire x1="144.78" y1="93.98" x2="160.02" y2="93.98" width="0.1524" layer="91"/>
-<wire x1="160.02" y1="93.98" x2="160.02" y2="101.6" width="0.1524" layer="91"/>
-<pinref part="Q21" gate="G$1" pin="E"/>
-<wire x1="160.02" y1="101.6" x2="154.94" y2="101.6" width="0.1524" layer="91"/>
-</segment>
-</net>
 <net name="N$17" class="0">
 <segment>
@@
 <net name="N$223" class="0">
 <segment>
-<pinref part="Q74" gate="G$1" pin="B"/>
-<wire x1="332.74" y1="106.68" x2="327.66" y2="106.68" width="0.1524" layer="91"/>
-<pinref part="R90" gate="G$1" pin="1"/>
-<wire x1="327.66" y1="111.76" x2="327.66" y2="106.68" width="0.1524" layer="91"/>
-<junction x="327.66" y="106.68"/>
-<wire x1="327.66" y1="106.68" x2="327.66" y2="96.52" width="0.1524" layer="91"/>
-<wire x1="327.66" y1="96.52" x2="337.82" y2="96.52" width="0.1524" layer="91"/>
 <pinref part="R78" gate="G$1" pin="2"/>
 <wire x1="332.74" y1="60.96" x2="332.74" y2="63.5" width="0.1524" layer="91"/>
@@
 <wire x1="332.74" y1="63.5" x2="337.82" y2="63.5" width="0.1524" layer="91"/>
 <junction x="337.82" y="63.5"/>
-<wire x1="337.82" y1="96.52" x2="337.82" y2="86.36" width="0.1524" layer="91"/>
+<wire x1="337.82" y1="101.6" x2="337.82" y2="86.36" width="0.1524" layer="91"/>
 <junction x="337.82" y="86.36"/>
+<pinref part="Q74" gate="G$1" pin="E"/>
 </segment>
 </net>
@@
 <junction x="259.08" y="35.56"/>
 <pinref part="Q81" gate="G$1" pin="B"/>
-</segment>
-</net>
-<net name="N$231" class="0">
-<segment>
-<pinref part="RV3" gate="G$1" pin="E"/>
-<wire x1="327.66" y1="91.44" x2="327.66" y2="93.98" width="0.1524" layer="91"/>
-<wire x1="327.66" y1="93.98" x2="342.9" y2="93.98" width="0.1524" layer="91"/>
-<wire x1="342.9" y1="93.98" x2="342.9" y2="101.6" width="0.1524" layer="91"/>
-<pinref part="Q74" gate="G$1" pin="E"/>
-<wire x1="342.9" y1="101.6" x2="337.82" y2="101.6" width="0.1524" layer="91"/>
 </segment>
 </net>
@@
 </segment>
 </net>
+<net name="N$122" class="0">
+<segment>
+<pinref part="Q74" gate="G$1" pin="B"/>
+<wire x1="332.74" y1="106.68" x2="327.66" y2="106.68" width="0.1524" layer="91"/>
+<pinref part="R90" gate="G$1" pin="1"/>
+<wire x1="327.66" y1="111.76" x2="327.66" y2="106.68" width="0.1524" layer="91"/>
+<pinref part="RV3" gate="G$1" pin="E"/>
+<wire x1="327.66" y1="106.68" x2="327.66" y2="91.44" width="0.1524" layer="91"/>
+<junction x="327.66" y="106.68"/>
+</segment>
+</net>
+<net name="N$1" class="0">
+<segment>
+<pinref part="Q21" gate="G$1" pin="B"/>
+<wire x1="149.86" y1="106.68" x2="144.78" y2="106.68" width="0.1524" layer="91"/>
+<pinref part="R30" gate="G$1" pin="1"/>
+<wire x1="144.78" y1="111.76" x2="144.78" y2="106.68" width="0.1524" layer="91"/>
+<pinref part="RV1" gate="G$1" pin="E"/>
+<wire x1="144.78" y1="106.68" x2="144.78" y2="91.44" width="0.1524" layer="91"/>
+<junction x="144.78" y="106.68"/>
+</segment>
+</net>
