File: THAT340/THAT340.brd (EAGLE design)
At the start: 10.1 x 20.3 mm, 5 parts, among them Q1 2SC1815, Q2 2SC1815, Q3 2SA1015, Q4 2SA1015

Commit message: VCFA2
Parts:
- moved Q2 1.00 mm to (5.08, 15.5)
- moved Q1 1.00 mm to (5.08, 13.0)
- moved Q3 1.00 mm to (5.08, 2.81)
- moved Q4 1.00 mm to (5.08, 5.35)
- moved U$1 1.00 mm to (8.89, 1.54)
Other:
- board size 10.1 x 20.3 mm -> 10.1 x 18.3 mm
- board text added: "THAT 340"
- board text removed: "THAT340"
