File: UbalToBal/UBTB_MIX.brd (EAGLE design)
At the start: 91.3 x 45 mm, 112 parts, among them IC1 OPA627U, IC2 OPA627U, Q26 BC847CSMD, Q29 BC857CSMD, Q30 BC847CSMD, Q31 BC847CSMD, Q32 BC847CSMD, Q33 BC857CSMD, Q34 BC857CSMD, Q35 BC857CSMD, Q36 BC857CSMD, Q37 BC847CSMD, Q38 BC847CSMD, Q39 BC847CSMD, Q40 BC857CSMD, Q41 BC857CSMD, X1 CON-PHOENIX-508_MKDSN1,5/3-5,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, X2 CON-PHOENIX-508_MKDSN1,5/3-5,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, X3 CON-PHOENIX-508_MKDSN1,5/2-5,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, X4 CON-PHOENIX-508_MKDSN1,5/2-5,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

Commit message: VCFA2
Parts:
- removed Q26, Q30, Q31, Q32, Q37, Q38, Q39: BC847CSMD, transistor-npn:SOT23
- removed Q29, Q33, Q34, Q35, Q36, Q40, Q41: BC857CSMD, transistor-pnp:SOT23-BEC
- removed R50, R52, R53, R54, R55, R56, R57, R58: (no value), Vwvwbg:MINI_MELF-0204W
- added Q17, Q18: (no value), Vwvwbg:TRANSISTOR_SOT23-BEC
- added U$1: LSK489SOP-6, Vwvwbg:SOT-23-6
- added U$2, U$3: LS3250, Vwvwbg:SOT-23-6
- added U$4: LSK689, Vwvwbg:SOT-23-6
- added U$5, U$6: LS3550, Vwvwbg:SOT-23-6
- C10, C7, C8, C9: device Vwvwbg:PANASONIC_E -> Vwvwbg:PANASONIC_F
- LED1, LED2, LED3, LED4, LED5, LED6, LED7, LED8: device led:CHIPLED_1206 -> Vwvwbg:LED_SML1206
- moved LED3 93.2 mm to (36.5, -52.5), flipped to the bottom, turned to 270 degrees
- moved R43 93.2 mm to (34.0, -52.5), flipped to the bottom, turned to 270 degrees
- moved R36 92.9 mm to (33.0, -52.5), turned to 270 degrees
- moved LED2 92.3 mm to (35.5, -52.5), turned to 270 degrees
- moved R35 91.9 mm to (38.0, -52.5), turned to 270 degrees
- moved R45 86.9 mm to (39.0, -52.5), flipped to the bottom
- moved R34 78.2 mm to (35.5, -43.5), turned to 0 degrees
- moved R33 69.7 mm to (31.5, -39.5), turned to 270 degrees
- moved R38 68.0 mm to (40.0, -42.5), turned to 90 degrees
- moved R40 59.9 mm to (32.8, -32.5), turned to 180 degrees
- moved R39 58.0 mm to (38.0, -32.5), turned to 0 degrees
- moved R42 53.9 mm to (32.8, -30.0), turned to 0 degrees
- moved R41 51.8 mm to (38.0, -30.0), turned to 180 degrees
- moved R37 44.7 mm to (39.5, -20.5)
- moved R32 44.1 mm to (31.5, -23.5), turned to 270 degrees
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Connections:
- removed net N$105: Q29.E, R35.1
- removed net N$106: Q40.E, R36.1
- new net N$2: R35.1, U$5.2
- new net N$23: R36.1, U$5.5
- net BOUT+: no longer R50.1, R52.1, R53.2, R54.2
- net BOUT-: no longer R55.1, R56.1, R57.2, R58.2
- net IN+: now also U$1.1, U$4.1, X3.1; no longer Q35.B, Q39.1, X4.1
- net IN-: now also U$1.4, U$4.4, X4.1; no longer Q34.B, Q38.1, X3.1
- net N$101: now also U$6.1, U$6.3; no longer Q33.B, Q41.B
- net N$102: now also U$1.2, U$5.4, U$6.5; no longer Q29.C, Q33.E, Q39.3
- net N$103: now also U$5.1, U$5.3; no longer Q29.B, Q40.B
- net N$104: now also U$1.5, U$5.6, U$6.2; no longer Q38.3, Q40.C, Q41.E
- net N$108: now also Q18.B; no longer Q36.B
- net N$109: now also Q18.E; no longer Q36.E
- net N$110: now also Q18.C; no longer Q36.C
- net N$111: now also U$4.6; no longer Q34.E
- net N$112: now also U$4.3; no longer Q35.E
- net N$115: now also U$1.3; no longer Q39.2
- net N$116: now also U$1.6; no longer Q38.2
- net N$117: now also Q17.C; no longer Q26.3
- net N$118: now also Q17.E; no longer Q26.2
- net N$119: now also Q17.B; no longer Q26.1
- net N$14: no longer R50.2
- net N$18: no longer R53.1
- net N$20: no longer R52.2
- net N$21: no longer R54.1
- net N$38: no longer R55.2
- net N$39: no longer R58.1
- net N$41: no longer R56.2
- net N$42: no longer R57.1
- net N$93: now also U$3.5; no longer Q30.2
- net N$94: now also U$3.2; no longer Q31.2
- net N$95: now also U$2.2, U$3.4, U$4.5; no longer Q31.3, Q32.2, Q34.C
- net N$96: now also U$2.5, U$3.6, U$4.2; no longer Q30.3, Q35.C, Q37.2
- net N$97: now also U$3.1, U$3.3; no longer Q30.1, Q31.1
- net N$98: now also U$2.1, U$2.3; no longer Q32.1, Q37.1
- net UOUT+: now also U$2.6, U$6.6; no longer Q33.C, Q37.3
- net UOUT-: now also U$2.4, U$6.4; no longer Q32.3, Q41.C
Routing:
- net V-: track 190.6 -> 5.35 mm, vias 5 -> 0
- net V+: track 187.2 -> 7.81 mm, vias 4 -> 0
- net IN-: track 68.5 -> 11.3 mm, vias 1 -> 0
- net IN+: track 65.2 -> 11.3 mm, vias 1 -> 0
- net BOUT-: track 45.4 -> 0.00 mm
- net BOUT+: track 44.5 -> 0.00 mm
- net N$9: track 33.4 -> 0.00 mm, vias 2 -> 0
- net N$30: track 28.7 -> 0.00 mm, vias 2 -> 0
- net N$12: track 24.4 -> 0.00 mm, vias 2 -> 0
- net N$33: track 21.2 -> 0.00 mm, vias 2 -> 0
- net N$10: track 20.2 -> 0.00 mm
- net N$29: track 19.6 -> 0.00 mm
- net UOUT-: track 41.2 -> 23.4 mm
- net N$22: track 15.2 -> 0.00 mm
- net N$27: track 14.0 -> 0.00 mm
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Other:
- board text removed: "0.1uF"
- board text removed: "10"
- board text removed: "10K"
- board text removed: "10uF"
- board text removed: "1K"
- board text removed: "1K3"
- board text removed: "250"
- board text removed: "300"
- board text removed: "KG UBalToBal Mod by Vwvwbg"
- board text removed: "OP27"
- board text removed: "OUT- IN+ GND V+ V-"
- board text removed: "P"
- board text removed: "RED"
- board text removed: "V+ V- GND IN+ OUT-"
- board text removed: "V1.0"
