File: UbalToBal/UBTB_MIX.sch (EAGLE design)
At the start: 112 parts, among them IC1 OPA627U, IC2 OPA627U, Q26 BC847CSMD, Q29 BC857CSMD, Q30 BC847CSMD, Q31 BC847CSMD, Q32 BC847CSMD, Q33 BC857CSMD, Q34 BC857CSMD, Q35 BC857CSMD, Q36 BC857CSMD, Q37 BC847CSMD, Q38 BC847CSMD, Q39 BC847CSMD, Q40 BC857CSMD, Q41 BC857CSMD, X1 CON-PHOENIX-508_MKDSN1,5/3-5,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, X2 CON-PHOENIX-508_MKDSN1,5/3-5,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, X3 CON-PHOENIX-508_MKDSN1,5/2-5,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, X4 CON-PHOENIX-508_MKDSN1,5/2-5,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

Commit message: VCFA2
Parts:
- removed Q26, Q30, Q31, Q32, Q37, Q38, Q39: BC847CSMD, transistor-npn:BC847CSMD
- removed Q29, Q33, Q34, Q35, Q36, Q40, Q41: BC857CSMD, transistor-pnp:BC857CSMD
- removed R50, R52, R53, R54, R55, R56, R57, R58: (no value), Vwvwbg:R-EU_MELF0204W
- added Q17: (no value), Vwvwbg:TRANSISTOR_BC846-NPN-SOT23-BEC
- added Q18: (no value), Vwvwbg:TRANSISTOR_BC856B-PNP-SOT23-BEC
- added U$1: LSK489SOP-6, Vwvwbg:LSK489SOP-6
- added U$2, U$3: LS3250, Vwvwbg:LS3250
- added U$4: LSK689, Vwvwbg:LSK689
- added U$5, U$6: LS3550, Vwvwbg:LS3550
- C10, C7, C8, C9: device Vwvwbg:CPOL-EUE -> Vwvwbg:CPOL-EUF
- LED1, LED2, LED3, LED4, LED5, LED6, LED7, LED8: device led:LEDCHIPLED_1206 -> Vwvwbg:LEDVWV1206
Connections:
- removed net N$105: Q29.E, R35.1
- removed net N$106: Q40.E, R36.1
- new net N$2: R35.1, U$5G$2.E
- new net N$23: R36.1, U$5G$1.E
- net BOUT+: no longer R50.1, R52.1, R53.2, R54.2
- net BOUT-: no longer R55.1, R56.1, R57.2, R58.2
- net IN+: now also U$1G$1.G, U$4G$1.G, X3-1.KL; no longer Q35.B, Q39.B, X4-1.KL
- net IN-: now also U$1G$2.G, U$4G$2.G, X4-1.KL; no longer Q34.B, Q38.B, X3-1.KL
- net N$101: now also U$6G$1.B, U$6G$2.B; no longer Q33.B, Q41.B
- net N$102: now also U$1G$1.D, U$5G$2.C, U$6G$1.E; no longer Q29.C, Q33.E, Q39.C
- net N$103: now also U$5G$1.B, U$5G$2.B; no longer Q29.B, Q40.B
- net N$104: now also U$1G$2.D, U$5G$1.C, U$6G$2.E; no longer Q38.C, Q40.C, Q41.E
- net N$108: now also Q18.B; no longer Q36.B
- net N$109: now also Q18.E; no longer Q36.E
- net N$110: now also Q18.C; no longer Q36.C
- net N$111: now also U$4G$2.S; no longer Q34.E
- net N$112: now also U$4G$1.S; no longer Q35.E
- net N$115: now also U$1G$1.S; no longer Q39.E
- net N$116: now also U$1G$2.S; no longer Q38.E
- net N$117: now also Q17.C; no longer Q26.C
- net N$118: now also Q17.E; no longer Q26.E
- net N$119: now also Q17.B; no longer Q26.B
- net N$14: no longer R50.2
- net N$18: no longer R53.1
- net N$20: no longer R52.2
- net N$21: no longer R54.1
- net N$38: no longer R55.2
- net N$39: no longer R58.1
- net N$41: no longer R56.2
- net N$42: no longer R57.1
- net N$93: now also U$3G$1.E; no longer Q30.E
- net N$94: now also U$3G$2.E; no longer Q31.E
- net N$95: now also U$2G$2.E, U$3G$2.C, U$4G$2.D; no longer Q31.C, Q32.E, Q34.C
- net N$96: now also U$2G$1.E, U$3G$1.C, U$4G$1.D; no longer Q30.C, Q35.C, Q37.E
- net N$97: now also U$3G$1.B, U$3G$2.B; no longer Q30.B, Q31.B
- net N$98: now also U$2G$1.B, U$2G$2.B; no longer Q32.B, Q37.B
- net UOUT+: now also U$2G$1.C, U$6G$1.C; no longer Q33.C, Q37.C
- net UOUT-: now also U$2G$2.C, U$6G$2.C; no longer Q32.C, Q41.C
