File: power/KGFV/UCC/KGGR_UCCv2.brd (EAGLE design)
At the start: 104.1 x 64.4 mm, 91 parts, among them IC1 OPA134, IC2 OPA134, Q12 DN2540, Q4 MJW21194, Q5 MJE15031, Q7 MJW21193, Q8 DN2540, Q9 MJE15030, X2 MKDSN1,5/3-5,08, X6 MKDSN1,5/2-5,08, X7 MKDSN1,5/2-5,08

Commit message: VCFA2
Other:
- board text added: "Vout = Vref * [ 1 + (R1/R2) ]"
- board text removed: "Vout=Vref*[1+(R1/R2)]"
Changed lines of the file:
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@@
 <?xml version="1.0" encoding="utf-8"?>
 <!DOCTYPE eagle SYSTEM "eagle.dtd">
-<eagle version="8.5.2">
+<eagle version="9.4.2">
 <drawing>
 <settings>
@@
 <wire x1="104.12" y1="64.44" x2="0" y2="64.44" width="0" layer="20"/>
 <wire x1="0" y1="64.44" x2="0" y2="0" width="0" layer="20"/>
-<text x="40.005" y="46.99" size="1.27" layer="21" rot="R90">NPN=KSP42
+<text x="40.64" y="62.865" size="1.27" layer="21" rot="R180">NPN=KSP42
 PNP=KSP92
 Zener=Vout/2</text>
-<text x="2.54" y="35.56" size="1.27" layer="21" rot="R90">Vout=Vref*[1+(R1/R2)]</text>
-<text x="45.72" y="62.23" size="1.27" layer="21">AC-IN</text>
+<text x="2.54" y="34.29" size="1.27" layer="21" rot="R90">Vout = Vref * [ 1 + (R1/R2) ]</text>
+<text x="49.53" y="62.23" size="1.27" layer="21">AC-IN</text>
 <text x="56.515" y="1.27" size="1.27" layer="25" font="fixed">+</text>
 <text x="51.435" y="1.27" size="1.27" layer="25">G</text>
@@
 <param name="checkStop" value="0"/>
 <param name="checkValues" value="0"/>
+<param name="checkNames" value="1"/>
+<param name="checkWireStubs" value="1"/>
+<param name="checkPolygonWidth" value="0"/>
 <param name="useDiameter" value="13"/>
 <param name="maxErrors" value="50"/>
@@
 </signal>
 </signals>
+<mfgpreviewcolors>
+<mfgpreviewcolor name="soldermaskcolor" color="0xC8008000"/>
+<mfgpreviewcolor name="silkscreencolor" color="0xFFFEFEFE"/>
+<mfgpreviewcolor name="backgroundcolor" color="0xFF282828"/>
+<mfgpreviewcolor name="coppercolor" color="0xFFFFBF00"/>
+<mfgpreviewcolor name="substratecolor" color="0xFF786E46"/>
+</mfgpreviewcolors>
 </board>
 </drawing>
