File: VCFA/VCFAA_v2.brd (EAGLE design)
At the start: 200 x 88 mm, 383 parts, among them IC1 LTC2057HV, IC2 LTC2057HV, IC3 LTC2057HV, IC4 LTC2057HV, IC5 OPA827, IC6 OPA827, J1 22-27-2031-03, J2 22-27-2031-03, Q1 LSK689, Q10 KSA992, Q100 MOS_SMDTDSON-8, Q105 MOS_SMDTDSON-8, Q106 MOS_SMDTDSON-8, Q107 MOS_SMDTDSON-8, Q108 MOS_SMDTDSON-8, Q11 KSA992, Q12 KSC1845, Q13 KSC1845, Q14 KSA992, Q15 KSC1845, Q16 KSA992, Q17 KSC1845, Q18 KSA992, Q19 KSA992, Q2 KSA992, Q20 KSC1845, Q21 KSC1845, Q22 KSA992, Q23 KSC1845, Q24 KSA992, Q25 KSA992, Q26 KSA992, Q27 KSC1845, Q28 KSC1845, Q29 KSC1845, Q3 KSC1845, Q30 KSC1845, Q31 KSA992, Q32 KSA992, Q33 KSA992, Q34 KSC1845, Q35 KSA992, Q36 KSA992, Q37 KSC1845, Q38 KSC1845, Q39 KSA1220, Q4 LSK489, Q40 KSC2690, Q41 KSA992, Q42 KSC1845, Q43 KSA992, Q44 KSC1845, Q45 MJE15030, Q46 KSC1845, Q47 KSA992, Q48 KSC1845, Q49 KSA992, Q5 LS3550, Q50 MJL4281A, Q51 MJL4302A, Q52 KSA992, Q53 KSA992, Q54 KSC1845, Q55 KSC1845, Q56 KSC1845, Q57 KSC1845, Q58 KSA992, Q59 KSA992, Q6 LS3250, Q60 KSA992, Q61 KSC1845, Q62 KSA992, Q63 KSA992, Q64 KSC1845, Q65 KSC1845, Q66 KSA1220, Q67 KSC2690, Q68 KSA992, Q69 KSC1845, Q7 LS3250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

Commit message: 0703
Parts:
- removed C37, C38: 10000uF, Vwvwbg:EB35D-8.5
- removed C39, C42, C58, C60: 0.1uF, Vwvwbg:C050-045X075
- removed C40, C41, C47, C48, C53, C54: 10uF, Vwvwbg:C1206
- removed C43, C44, C45, C46, C49, C50: 0.1uF, Vwvwbg:C0805
- removed C51, C52: 47p, Vwvwbg:C0805
- removed C55, C56: 4.7uF, Vwvwbg:C050-075X075
- removed C57, C59: 47uF, Vwvwbg:C1206
- removed C61, C62, C64: (no value), Vwvwbg:C0805
- removed C63: 1n, Vwvwbg:C0805
- removed D13, D14: BZT55B10, Vwvwbg:SOD80C
- removed D15, D16: S1G, Vwvwbg:DO214AA
- removed D17, D18: LT1236-10, Vwvwbg:SO8
- removed D19, D20, D21, D22: LL4148, Vwvwbg:SOD80C
- removed IC5, IC6: OPA827, Vwvwbg:SOIC8
- removed J1, J2: 22-27-2031-03, con-molex:6410-03
- removed LED13, LED14, LED15, LED16: RED, Vwvwbg:LED_SML1206
- removed Q100, Q105, Q106, Q107, Q108, Q97, Q98, Q99: MOS_SMDTDSON-8, Vwvwbg:PG-TDSON-8
- removed Q79, Q82, Q84, Q86, Q87: KSC1845, Vwvwbg:TRANSISTOR_TO92-ECB_N
- removed Q80, Q81, Q83, Q85, Q88: KSA992, Vwvwbg:TRANSISTOR_TO92-ECB_P
- removed Q89: MJL4281A, Vwvwbg:TRANSISTOR_TO247_BCE_N
- removed Q90: MJL4302A, Vwvwbg:TRANSISTOR_TO247_BCE_P
- removed Q91, Q92: DN2540, Vwvwbg:TRANSISTOR_TO92-SGD_N
- removed R115, R116: 10k, Vwvwbg:MINI_MELF-0204W
- removed R117, R118, R125, R126: 1k, Vwvwbg:MINI_MELF-0204W
- removed R119, R122: 100, Vwvwbg:MINI_MELF-0204W
- removed R120, R121, R123, R124: 10, Vwvwbg:MINI_MELF-0204W
- removed R127, R128, R129, R130: 1.5k, Vwvwbg:MINI_MELF-0204W
- removed U$1, U$3: ACHS-712X, Vwvwbg:SO8
- removed U$2, U$4: LT4320MSOP, Vwvwbg:LT4320_MSOP
- removed X2, X3: (no value), Vwvwbg:KK-156-2
- moved H4 38.0 mm to (158.0, 81.0)
- moved H1 34.5 mm to (38.5, 4.00)
- moved H2 34.5 mm to (161.5, 4.00)
- moved H5 29.0 mm to (36.5, 84.0)
- moved H3 17.6 mm to (20.5, 86.5)
- moved C6 4.00 mm to (49.0, 14.5)
Connections:
- removed net AC1: Q100.5, Q100.6, Q100.7, Q100.8, Q100.TH, Q97.1, Q97.2, Q97.3, U$2.1, X3.2
- removed net AC2: Q98.1, Q98.2, Q98.3, Q99.5, Q99.6, Q99.7, Q99.8, Q99.TH, U$2.12, X3.1
- removed net AC3: Q105.1, Q105.2, Q105.3, Q108.5, Q108.6, Q108.7, Q108.8, Q108.TH, U$4.1, X2.2
- removed net AC4: Q106.1, Q106.2, Q106.3, Q107.5, Q107.6, Q107.7, Q107.8, Q107.TH, U$4.12, X2.1
- removed net D5V1: C64.1, J1.1, U$1.8
- removed net D5V2: C61.1, J2.1, U$3.8
- removed net DGND1: C63.2, C64.2, J1.3, U$1.5
- removed net DGND2: C61.2, C62.2, J2.3, U$3.5
- removed net N$1: Q79.C, Q81.B, Q81.C, Q83.B
- removed net N$100: C40.1, C43.1, D13.C, Q83.C, Q87.B
- removed net N$105: C40.2, C43.2, D13.A, R120.1
- removed net N$106: Q85.E, R120.2
- removed net N$107: Q79.E, R117.1
- removed net N$113: LED13.A, Q79.B, R115.2
- removed net N$114: Q80.E, R118.2
- removed net N$119: LED14.C, Q80.B, R116.1
- removed net N$120: Q86.E, R121.1
- removed net N$121: C41.1, C44.1, D14.C, R121.2
- removed net N$122: C41.2, C44.2, D14.A, Q84.C, Q88.B
- removed net N$123: Q80.C, Q82.B, Q82.C, Q84.B
- removed net N$124: Q84.E, R122.1
- removed net N$125: LED16.A, Q82.E
- removed net N$126: Q88.E, Q90.B
- removed net N$127: Q87.E, Q89.B
- removed net N$128: C51.1, IC6.6, R123.1
- removed net N$129: C52.1, IC5.6, R124.1
- removed net N$130: Q86.B, R124.2
- removed net N$131: Q85.B, R123.2
- removed net N$132: C51.2, C53.2, D19.A, D20.C, IC6.2, R127.1, R128.2
- removed net N$133: C47.1, C49.1, D17.6, D19.C, D20.A, IC6.3, Q91.G, R125.1
- removed net N$134: Q91.S, R125.2
- removed net N$135: C48.2, C50.2, D18.4, D21.A, D22.C, IC5.3, Q92.D
- removed net N$136: Q92.S, R126.2
- removed net N$137: C52.2, C54.1, D21.C, D22.A, IC5.2, R129.1, R130.2
- removed net N$143: C63.1, U$1.6
- removed net N$157: Q98.4, U$2.11
- removed net N$184: Q100.4, U$2.6
- removed net N$188: Q97.4, U$2.2
- removed net N$189: Q99.4, U$2.5
- removed net N$201: Q106.4, U$4.11
- removed net N$204: Q108.4, U$4.6
- removed net N$208: Q105.4, U$4.2
- removed net N$209: Q107.4, U$4.5
- removed net N$75: LED15.C, Q81.E
- removed net N$90: Q83.E, R119.2
- removed net N$91: C62.1, U$3.6
- removed net UV+: C57.1, Q97.5, Q97.6, Q97.7, Q97.8, Q97.TH, Q98.5, Q98.6, Q98.7, Q98.8, Q98.TH, U$1.1, U$1.2, U$2.9
- removed net UV+IN: C37.+, C42.2, C58.2, D15.C, LED15.A, Q87.C, Q89.C, R115.1, R119.1, U$1.3, U$1.4
- removed net UV-: C59.2, Q107.1, Q107.2, Q107.3, Q108.1, Q108.2, Q108.3, U$3.3, U$3.4, U$4.7, U$4.EXP
- removed net UV-IN: C38.-, C39.1, C60.1, D16.A, LED16.C, Q88.C, Q90.C, R116.2, R122.2, U$3.1, U$3.2
- removed net VS+: J1.2, U$1.7
- removed net VS-: J2.2, U$3.7
- net GND: no longer C37.-, C38.+, C39.2, C42.1, C45.1, C46.2, C47.2, C48.1, C49.2, C50.1, C55.1, C56.2, C57.2, C58.1, C59.1, C60.2, D17.4, D18.6, IC5.7, IC6.4, LED13.C, LED14.A, Q100.1, Q100.2, Q100.3, Q105.5, Q105.6, Q105.7, Q105.8, Q105.TH, Q106.5, Q106.6, Q106.7, Q106.8, Q106.TH, Q85.C, Q86.C, Q99.1, Q99.2, Q99.3, R117.2, R118.1, R128.1, R129.2, U$2.7, U$2.EXP, U$4.9
- net V+: no longer C45.2, C53.1, C55.2, D15.A, IC6.7, Q89.E, Q91.D, R127.2
- net V-: no longer C46.1, C54.2, C56.1, D16.C, IC5.4, Q90.E, Q92.G, R126.1, R130.1
Routing:
- net V-: track 491.7 -> 362.9 mm, vias 4 -> 3
- net V+: track 493.6 -> 393.9 mm, vias 9 -> 7
- net UV-IN: track 71.6 -> 0.00 mm
- net UV+IN: track 66.2 -> 0.00 mm
- net N$133: track 32.1 -> 0.00 mm, vias 1 -> 0
- net N$135: track 23.2 -> 0.00 mm, vias 1 -> 0
- net N$132: track 18.7 -> 0.00 mm, vias 1 -> 0
- net N$126: track 17.9 -> 0.00 mm
- net D5V2: track 17.6 -> 0.00 mm
- net UV+: track 17.0 -> 0.00 mm
- net N$105: track 16.8 -> 0.00 mm
- net VS-: track 16.0 -> 0.00 mm
- net N$137: track 15.8 -> 0.00 mm, vias 1 -> 0
- net N$122: track 15.6 -> 0.00 mm
- net N$127: track 14.6 -> 0.00 mm
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- removed copper zone on layer 1, net AC1
- removed copper zone on layer 1, net AC2
- removed copper zone on layer 16, net AC2
- removed copper zone on layer 1, net AC3
- removed copper zone on layer 16, net AC3
- removed copper zone on layer 1, net AC4
- removed copper zone on layer 1, net DGND1
- removed copper zone on layer 16, net DGND1
- removed copper zone on layer 1, net DGND2
- removed copper zone on layer 16, net DGND2
- removed copper zone on layer 1, net N$141
- removed copper zone on layer 16, net N$141
- removed copper zone on layer 1, net UV+
- removed copper zone on layer 1, net UV+IN
- removed copper zone on layer 1, net UV-
- removed copper zone on layer 1, net UV-IN
Other:
- board size 200 x 88 mm -> 167.5 x 88 mm
- board text removed: "0.1F"
- board text removed: "10000uF"
- board text removed: "10F"
- board text removed: "10V"
- board text removed: "10u"
- board text removed: "1k5"
- board text removed: "1uF"
- board text removed: "1uF 100V"
- board text removed: "2k4"
- board text removed: "4.7uF"
- board text removed: "47p"
- board text removed: "AC"
- board text removed: "ACHS 7122"
- board text removed: "B C F A II"
- board text removed: "GND S- 5V"
- board text removed: "LT1236-10"
- board text removed: "LT4320"
- board text removed: "MOS BSC031N06NS3 G"
- board text removed: "OPA828"
- board text removed: "V+"
- board text removed: "V-"
