File: VCFA/VCFAA_v2.sch (EAGLE design)
At the start: 383 parts, among them IC1 LTC2057HV, IC2 LTC2057HV, IC3 LTC2057HV, IC4 LTC2057HV, IC5 OPA827, IC6 OPA827, J1 22-27-2031-03, J2 22-27-2031-03, Q1 LSK689, Q10 KSA992, Q100 MOS_SMDTDSON-8, Q105 MOS_SMDTDSON-8, Q106 MOS_SMDTDSON-8, Q107 MOS_SMDTDSON-8, Q108 MOS_SMDTDSON-8, Q11 KSA992, Q12 KSC1845, Q13 KSC1845, Q14 KSA992, Q15 KSC1845, Q16 KSA992, Q17 KSC1845, Q18 KSA992, Q19 KSA992, Q2 KSA992, Q20 KSC1845, Q21 KSC1845, Q22 KSA992, Q23 KSC1845, Q24 KSA992, Q25 KSA992, Q26 KSA992, Q27 KSC1845, Q28 KSC1845, Q29 KSC1845, Q3 KSC1845, Q30 KSC1845, Q31 KSA992, Q32 KSA992, Q33 KSA992, Q34 KSC1845, Q35 KSA992, Q36 KSA992, Q37 KSC1845, Q38 KSC1845, Q39 KSA1220, Q4 LSK489, Q40 KSC2690, Q41 KSA992, Q42 KSC1845, Q43 KSA992, Q44 KSC1845, Q45 MJE15030, Q46 KSC1845, Q47 KSA992, Q48 KSC1845, Q49 KSA992, Q5 LS3550, Q50 MJL4281A, Q51 MJL4302A, Q52 KSA992, Q53 KSA992, Q54 KSC1845, Q55 KSC1845, Q56 KSC1845, Q57 KSC1845, Q58 KSA992, Q59 KSA992, Q6 LS3250, Q60 KSA992, Q61 KSC1845, Q62 KSA992, Q63 KSA992, Q64 KSC1845, Q65 KSC1845, Q66 KSA1220, Q67 KSC2690, Q68 KSA992, Q69 KSC1845, Q7 LS3250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

Commit message: 0703
Parts:
- removed C37, C38: 10000uF, Vwvwbg:CPOL-EU
- removed C39, C42, C58, C60: 0.1uF, Vwvwbg:C-EU050-045X075
- removed C40, C41, C47, C48, C53, C54: 10uF, Vwvwbg:C-EUC1206
- removed C43, C44, C45, C46, C49, C50: 0.1uF, Vwvwbg:C-EUC0805
- removed C51, C52: 47p, Vwvwbg:C-EUC0805
- removed C55, C56: 4.7uF, Vwvwbg:C-EU050-075X075
- removed C57, C59: 47uF, Vwvwbg:C-EUC1206
- removed C61, C62, C64: (no value), Vwvwbg:C-EUC0805
- removed C63: 1n, Vwvwbg:C-EUC0805
- removed D13, D14: BZT55B10, Vwvwbg:DIODE-SOD80C
- removed D15, D16: S1G, Vwvwbg:DIODE-DO214AA
- removed D17, D18: LT1236-10, Vwvwbg:LINEAR-TECHNOLOGY_LT1021-VSO-8
- removed D19, D20, D21, D22: LL4148, Vwvwbg:DIODE-SOD80C
- removed IC5, IC6: OPA827, Vwvwbg:LT1037CS8
- removed J1, J2: 22-27-2031-03, con-molex:22-27-2031-03
- removed LED13, LED14, LED15, LED16: RED, Vwvwbg:LEDVWV1206
- removed Q100, Q105, Q106, Q107, Q108, Q97, Q98, Q99: MOS_SMDTDSON-8, Vwvwbg:MOS_SMDTDSON-8
- removed Q79, Q82, Q84, Q86, Q87: KSC1845, Vwvwbg:BJT_NPNKSC1845
- removed Q80, Q81, Q83, Q85, Q88: KSA992, Vwvwbg:BJT_PNPKSA992
- removed Q89: MJL4281A, Vwvwbg:BJT_NPNMJL4281
- removed Q90: MJL4302A, Vwvwbg:BJT_PNPMJL4302
- removed Q91, Q92: DN2540, Vwvwbg:DN2540
- removed R115, R116: 10k, Vwvwbg:R-EU_MELF0204W
- removed R117, R118, R125, R126: 1k, Vwvwbg:R-EU_MELF0204W
- removed R119, R122: 100, Vwvwbg:R-EU_MELF0204W
- removed R120, R121, R123, R124: 10, Vwvwbg:R-EU_MELF0204W
- removed R127, R128, R129, R130: 1.5k, Vwvwbg:R-EU_MELF0204W
- removed U$1, U$3: ACHS-712X, Vwvwbg:ACHS-712X
- removed U$2, U$4: LT4320MSOP, Vwvwbg:LT4320MSOP
- removed X2, X3: (no value), Vwvwbg:KK-156-2
Connections:
- removed net AC1: Q100.D, Q97.S, U$2.1_IN2, X3-2.S
- removed net AC2: Q98.S, Q99.D, U$2.8_IN1, X3-1.S
- removed net AC3: Q105.S, Q108.D, U$4.1_IN2, X2-2.S
- removed net AC4: Q106.S, Q107.D, U$4.8_IN1, X2-1.S
- removed net D5V1: C64.1, J1-1.S, U$1.VDD
- removed net D5V2: C61.1, J2-1.S, U$3.VDD
- removed net DGND1: C63.2, C64.2, J1-3.S, U$1.GND
- removed net DGND2: C61.2, C62.2, J2-3.S, U$3.GND
- removed net N$1: Q79.C, Q81.B, Q81.C, Q83.B
- removed net N$100: C40.1, C43.1, D13.C, Q83.C, Q87.B
- removed net N$105: C40.2, C43.2, D13.A, R120.1
- removed net N$106: Q85.E, R120.2
- removed net N$107: Q79.E, R117.1
- removed net N$113: LED13.A, Q79.B, R115.2
- removed net N$114: Q80.E, R118.2
- removed net N$119: LED14.C, Q80.B, R116.1
- removed net N$120: Q86.E, R121.1
- removed net N$121: C41.1, C44.1, D14.C, R121.2
- removed net N$122: C41.2, C44.2, D14.A, Q84.C, Q88.B
- removed net N$123: Q80.C, Q82.B, Q82.C, Q84.B
- removed net N$124: Q84.E, R122.1
- removed net N$125: LED16.A, Q82.E
- removed net N$126: Q88.E, Q90.B
- removed net N$127: Q87.E, Q89.B
- removed net N$128: C51.1, IC6.OUT, R123.1
- removed net N$129: C52.1, IC5.OUT, R124.1
- removed net N$130: Q86.B, R124.2
- removed net N$131: Q85.B, R123.2
- removed net N$132: C51.2, C53.2, D19.A, D20.C, IC6.-IN, R127.1, R128.2
- removed net N$133: C47.1, C49.1, D17.OUT, D19.C, D20.A, IC6.+IN, Q91.G, R125.1
- removed net N$134: Q91.S, R125.2
- removed net N$135: C48.2, C50.2, D18.GND, D21.A, D22.C, IC5.+IN, Q92.D
- removed net N$136: Q92.S, R126.2
- removed net N$137: C52.2, C54.1, D21.C, D22.A, IC5.-IN, R129.1, R130.2
- removed net N$143: C63.1, U$1.FILTER
- removed net N$157: Q98.G, U$2.7_TG1
- removed net N$184: Q100.G, U$2.4_BG1
- removed net N$188: Q97.G, U$2.2_TG2
- removed net N$189: Q99.G, U$2.3_BG2
- removed net N$201: Q106.G, U$4.7_TG1
- removed net N$204: Q108.G, U$4.4_BG1
- removed net N$208: Q105.G, U$4.2_TG2
- removed net N$209: Q107.G, U$4.3_BG2
- removed net N$75: LED15.C, Q81.E
- removed net N$90: Q83.E, R119.2
- removed net N$91: C62.1, U$3.FILTER
- removed net UV+: C57.1, Q97.D, Q98.D, U$1.I+, U$2.6_OUTP
- removed net UV+IN: C37.+, C42.2, C58.2, D15.C, LED15.A, Q87.C, Q89.C, R115.1, R119.1, U$1.I-
- removed net UV-: C59.2, Q107.S, Q108.S, U$3.I-, U$4.5_OUTN
- removed net UV-IN: C38.-, C39.1, C60.1, D16.A, LED16.C, Q88.C, Q90.C, R116.2, R122.2, U$3.I+
- removed net VS+: J1-2.S, U$1.VOUT
- removed net VS-: J2-2.S, U$3.VOUT
- net GND: no longer C37.-, C38.+, C39.2, C42.1, C45.1, C46.2, C47.2, C48.1, C49.2, C50.1, C55.1, C56.2, C57.2, C58.1, C59.1, C60.2, D17.GND, D18.OUT, IC5.V+, IC6.V-, LED13.C, LED14.A, Q100.S, Q105.D, Q106.D, Q85.C, Q86.C, Q99.S, R117.2, R118.1, R128.1, R129.2, U$2.5_OUTN, U$4.6_OUTP
- net V+: no longer C45.2, C53.1, C55.2, D15.A, IC6.V+, Q89.E, Q91.D, R127.2
- net V-: no longer C46.1, C54.2, C56.1, D16.C, IC5.V-, Q90.E, Q92.G, R126.1, R130.1
