File: pi/pi.sch (EAGLE design)
At the start: 0 parts

Commit message: 0703
Parts:
- added C1, C10, C11, C12, C13, C14, C15, C16, C17, C18, C19, C2, C3, C4, C5, C6, C7, C8, C9: 0.1uF, Vwvwbg:C-EUC0603K
- added J1: HFJ11-1G02E-L12RL, Vwvwbg:HFJ11-1G02E-L12RL
- added PCB1: RPI_COMPUTE, Vwvwbg:RPI_COMPUTE
- added R1, R2, R3, R4, R5, R6, R7, R8: (no value), Vwvwbg:R-EU_MELF0204R
- added R10: 12k, Vwvwbg:R-EU_MELF0204R
- added R11: 10k, Vwvwbg:R-EU_MELF0204R
- added R12, R13, R14, R16: BEAD, Vwvwbg:R-EU_MELF0204R
- added R15: 0, Vwvwbg:R-EU_MELF0204R
- added R9: 8.06k, Vwvwbg:R-EU_MELF0204R
- added U$1: DD21, Vwvwbg:DD21
- added U$2: IRM-15-5, Vwvwbg:IRM-15-5
- added U1: LAN7500I-ABZJ-TR, Vwvwbg:LAN7500I-ABZJ-TR
Connections:
- new net +1.2V: C19.1, C4.1, C5.1, C6.1, C7.1, C8.1, C9.1, R12.2, R13.2, R16.2, U1.VDD12BIAS, U1.VDD12CORE
- new net +2.5V: C15.1, C16.1, C17.1, C18.1, U1.VDDVARIO
- new net +2.5VA: J1.VCC, R1.2, R2.2, R3.2, R4.2, R5.2, R6.2, R7.2, R8.2
- new net +3.3V: R14.1
- new net CGND: J1.GND, R15.1
- new net GND1: C1.2, C10.2, C11.2, C12.2, C13.2, C14.2, C15.2, C16.2, C17.2, C18.2, C19.2, C2.2, C3.2, C4.2, C5.2, C6.2, C7.2, C8.2, C9.2, R10.2, R15.2, R9.1, U1.VSS
- new net N$1: R9.2, U1.ETHRBIAS
- new net N$2: R10.1, U1.USBRBIAS
- new net N$3: R11.1, U1.VBUS_DET
- new net TD0_N: J1.TD0-, R1.1, U1.TR0N
- new net TD0_P: J1.TD0+, R2.1, U1.TR0P
- new net TD1_N: J1.TD1-, R3.1, U1.TR1N
- new net TD1_P: J1.TD1+, R4.1, U1.TR1P
- new net TD2_N: J1.TD2-, R5.1, U1.TR2N
- new net TD2_P: J1.TD2+, R6.1, U1.TR2P
- new net TD3_N: J1.TD3-, R7.1, U1.TR3N
- new net TD3_P: J1.TD3+, R8.1, U1.TR3P
- new net USB_N: PCB1.167/USB_DM**, U1.USBDM
- new net USB_P: PCB1.165/USB_DP**, U1.USBDP
- new net VDD12A: C10.1, C11.1, C12.1, C13.1, C14.1, R16.1, U1.VDD12A
- new net VDD12PLL: C2.1, R13.1, U1.VDD12PLL
- new net VDD12USBPLL: C1.1, R12.1, U1.VDD12USBPLL
- new net VDD33A: C3.1, R11.2, R14.2, U1.VDD33A
